File: Heatplate_v2.0/Heatplate_v2.0.kicad_pcb (KiCad board)
At the start: 2 copper layers, 100 x 121 mm, 58 parts, among them J1 Barrel_Jack_Switch, J4 1x8 2.54mm female, J5 1x8 2.54mm male, Q1 WSP4409A, Q2 IRLR8726TRPBF, Q3 SS8050, SW1 SW_Push, SW2 SW_Push, U1 ATMEGA4809-AFR, U2 AMS1117-5.0

Commit message: Minor fixes
Parts:
- added mouse-bite-5mm-slot: VAL**, Library:mouse-bite-5mm-slot, F.Cu at (88.9, 86.3)
- added mouse-bite-5mm-slot: VAL**, Library:mouse-bite-5mm-slot, F.Cu at (135.0, 86.3)
- moved J5 13.2 mm to (101.2, 91.1)
- moved H3 13.2 mm to (63.5, 164.3)
- moved H4 13.2 mm to (156.5, 164.3)
- moved LOGO1 13.2 mm to (64.5, 120.8)
- moved H7 13.2 mm to (63.5, 92.2)
- moved H8 13.2 mm to (156.5, 92.3)
Routing:
- net unconnected-(U1-PF2-Pad36): track 22.8 -> 0.00 mm, vias 3 -> 0
- net /TDATA_D: track 29.6 -> 25.4 mm, vias 3 -> 2
- net HEATPLATE: track 3339.5 -> 3335.4 mm
- net +5V: track 101.5 -> 98.3 mm, vias 1 -> 0
Other:
- board size 100 x 121 mm -> 100 x 107.8 mm
- board text added: "Ver 2.0"
- board text removed: "Ver 1.1"
